File: hardware/s88nsniffer/s88nsniffer.kicad_sch (KiCad schematic)
At the start: 20 parts, among them J101 RJ45, J102 RJ45, J103 Conn_01x09_Pin, J108 Conn_01x03_Pin, J109 Conn_01x02_Pin, U101 74HC14, U102 TSR_1-2490, U104 ULN2803A

Commit message: add component values add some info on the schematic fixed a nr of pcb layout issues
Parts:
- C101, C103: value C -> 100n
- C102: value C_Polarized -> 470u
- R101, R102, R103: value R -> 47R
Connections:
- no-connect marks 12 -> 10
Other:
- note added: "A6 AND A7 CAN ONLY BE USED AS ANALOG INPUT ON NANO V3"
- note added: "The 74HC14 stages aren't strictly necessary. They sharpen the S88 signals (LOAD, CLOCK, DATA) with Schmitt-trigger inputs and help reduce noise."
Changed lines of the file:
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@@
 	(generator_version "9.0")
 	(paper "A4")
+	(text "The 74HC14 stages aren't strictly necessary.\nThey sharpen the S88 signals (LOAD, CLOCK, DATA) \nwith Schmitt-trigger inputs and help reduce noise."
+		(exclude_from_sim no)
+		(at 83.82 116.84 0)
+		(effects
+			(font
+				(size 1.27 1.27)
+			)
+			(justify left)
+		)
+	)
+	(text "A6 AND A7 CAN ONLY BE \nUSED AS ANALOG INPUT ON NANO V3"
+		(exclude_from_sim no)
+		(at 208.534 119.634 0)
+		(effects
+			(font
+				(size 1.27 1.27)
+			)
+		)
+	)
 	(junction
 		(at 170.18 114.3)
@@
 	)
 	(junction
-		(at 104.14 107.95)
-		(diameter 0)
-		(color 0 0 0 0)
-	)
-	(junction
 		(at 149.86 52.07)
 		(diameter 0)
@@
 	)
 	(no_connect
-		(at 104.14 107.95)
-	)
-	(no_connect
 		(at 157.48 104.14)
 	)
@@
 	)
 	(no_connect
-		(at 125.73 92.71)
-	)
-	(no_connect
 		(at 172.72 60.96)
 	)
@@
 	(wire
 		(pts
-			(xy 102.87 107.95) (xy 104.14 107.95)
+			(xy 104.14 107.95) (xy 111.76 107.95)
 		)
 		(stroke
@@
 		)
 	)
-	(wire
-		(pts
-			(xy 104.14 107.95) (xy 111.76 107.95)
-		)
-		(stroke
-			(width 0)
-			(type default)
-		)
-	)
 	(label "clock"
 		(at 137.16 76.2 0)
@@
 			)
 		)
-		(property "Value" "C"
+		(property "Value" "100n"
 			(at 121.92 45.7199 0)
 			(effects
@@
 			)
 		)
-		(property "Value" "R"
+		(property "Value" "47R"
 			(at 74.93 104.14 90)
 			(effects
@@
 			)
 		)
-		(property "Value" "R"
+		(property "Value" "47R"
 			(at 74.93 88.9 90)
 			(effects
@@
 			)
 		)
-		(property "Value" "C_Polarized"
+		(property "Value" "470u"
 			(at 133.35 44.8309 0)
 			(effects
@@
 			)
 		)
-		(property "Value" "R"
+		(property "Value" "47R"
 			(at 73.66 72.39 90)
 			(effects
@@
 			)
 		)
-		(property "Value" "C"
+		(property "Value" "100n"
 			(at 210.82 34.2899 0)
 			(effects

Commit message: BOM details updated
Parts:
- J101: value RJ45 -> RJ45C5 T1U 2.8N4N TY; MFR (none) -> WEIDMULLER; MPN (none) -> 1455240000
- J102: value RJ45 -> RJ45C5 T1U 2.8N4N TY; MFR (none) -> Weidmuller; MPN (none) -> 1455240000
- J103: value Conn_01x09_Pin -> B9B-PH-K-S
- J108: value Conn_01x03_Pin -> B3B-PH-K-S; MFR (none) -> JST; MPN (none) -> B3B-PH-K-S
Other:
- note added: "Weidmuller 1455240000"
Changed lines of the file:
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@@
 		)
 	)
+	(text "\nWeidmuller \n1455240000\n"
+		(exclude_from_sim no)
+		(at 22.098 67.31 0)
+		(effects
+			(font
+				(size 1.27 1.27)
+			)
+		)
+	)
+	(text "\nWeidmuller \n1455240000\n"
+		(exclude_from_sim no)
+		(at 98.806 58.674 0)
+		(effects
+			(font
+				(size 1.27 1.27)
+			)
+		)
+	)
 	(text "A6 AND A7 CAN ONLY BE \nUSED AS ANALOG INPUT ON NANO V3"
 		(exclude_from_sim no)
@@
 		(on_board yes)
 		(dnp no)
-		(fields_autoplaced yes)
 		(property "Reference" "J103"
 			(at 275.59 92.7099 0)
@@
 			)
 		)
-		(property "Value" "Conn_01x09_Pin"
-			(at 275.59 95.2499 0)
+		(property "Value" "B9B-PH-K-S"
+			(at 261.112 105.918 0)
 			(effects
 				(font
@@
 		(on_board yes)
 		(dnp no)
-		(fields_autoplaced yes)
 		(property "Reference" "J101"
 			(at 21.59 38.1 0)
@@
 			)
 		)
-		(property "Value" "RJ45"
-			(at 21.59 40.64 0)
+		(property "Value" "RJ45C5 T1U 2.8N4N TY"
+			(at 28.956 40.894 0)
 			(effects
 				(font
@@
 			)
 		)
+		(property "MFR" "WEIDMULLER"
+			(at 21.59 55.88 0)
+			(effects
+				(font
+					(size 1.27 1.27)
+				)
+				(hide yes)
+			)
+		)
+		(property "MPN" "1455240000"
+			(at 21.59 55.88 0)
+			(effects
+				(font
+					(size 1.27 1.27)
+				)
+				(hide yes)
+			)
+		)
 		(pin "3"
 		)
@@
 			)
 		)
-		(property "Value" "RJ45"
-			(at 83.82 40.64 0)
+		(property "Value" "RJ45C5 T1U 2.8N4N TY"
+			(at 79.248 40.64 0)
 			(effects
 				(font
@@
 			)
 		)
+		(property "MFR" "Weidmuller"
+			(at 83.82 55.88 0)
+			(effects
+				(font
+					(size 1.27 1.27)
+				)
+				(hide yes)
+			)
+		)
+		(property "MPN" "1455240000"
+			(at 83.82 55.88 0)
+			(effects
+				(font
+					(size 1.27 1.27)
+				)
+				(hide yes)
+			)
+		)
 		(pin "3"
 		)
@@
 		(dnp no)
 		(property "Reference" "J108"
-			(at 85.344 32.004 0)
+			(at 109.474 41.656 0)
 			(effects
 				(font
@@
 			)
 		)
-		(property "Value" "Conn_01x03_Pin"
-			(at 87.122 35.052 0)
+		(property "Value" "B3B-PH-K-S"
+			(at 105.41 34.036 0)
 			(effects
 				(font
@@
 			(at 93.98 44.45 0)
 			(effects
+				(font
+					(size 1.27 1.27)
+				)
+				(hide yes)
+			)
+		)
+		(property "MFR" "JST"
+			(at 93.98 44.45 0)
+			(effects
+				(font
+					(size 1.27 1.27)
+				)
+				(hide yes)
+			)
+		)
+		(property "MPN" "B3B-PH-K-S"
+			(at 93.98 44.45 0)
+			(effects
